File: Anduril USB Hub.kicad_pcb (KiCad board)
At the start: 2 copper layers, 30 parts, among them J1 USB C 2.0, Upstream, J2 USB A, Port 1, J3 USB A, Port 2, J4 USB C 2.0, Port 3, U1 USB4604-1080HN, U2 USBLC6-2SC6, U3 USBLC6-2SC6, U4 USBLC6-2SC6, Y1 24M

Commit message: blah blah comment
Parts:
- added R4: 5k, Resistor_SMD:R_0805_2012Metric, F.Cu at (208.3, 47.0)
- Y1: value 24M -> Crystal_GND24; footprint Crystal:Crystal_SMD_3225-4Pin_3.2x2.5mm -> Crystal:Crystal_SMD_0603-4Pin_6.0x3.5mm
- moved RESET1 77.0 mm to (204.9, 65.7)
- moved R2 77.0 mm to (207.6, 58.2)
- moved C1 69.2 mm to (142.4, 75.6), turned to -90 degrees
- moved F3 65.2 mm to (194.4, 75.9), turned to 90 degrees
- moved U3 64.7 mm to (199.2, 75.8), turned to 90 degrees
- moved J3 63.7 mm to (195.8, 83.3)
- moved J2 61.6 mm to (141.9, 83.4)
- moved U2 61.6 mm to (145.3, 75.6), turned to 90 degrees
- moved C4 57.2 mm to (196.5, 75.9), turned to -90 degrees
- moved R1 42.1 mm to (182.8, 42.9)
- moved R3 41.2 mm to (182.8, 45.0)
- moved F4 33.3 mm to (168.0, 80.6), turned to 90 degrees
- moved F2 28.5 mm to (140.2, 75.6), turned to 90 degrees
- moved C3 24.5 mm to (156.1, 44.3), turned to 90 degrees
- moved Y1 24.3 mm to (151.6, 44.2), turned to 0 degrees
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Connections:
- net VDDCR12 renamed VDD12
- C5 pad 1: VCC -> +5V
- C6 pad 1: VCC -> +5V
- C7 pad 1: VCC -> +5V
- J1 pad A6: D+ UP -> UP D+
- J1 pad A7: D- UP -> UP D-
- J1 pad B6: D+ UP -> UP D+
- J1 pad B7: D- UP -> UP D-
- U3 pad 4: P2 D- -> P3 D-
- U3 pad 6: P2 D+ -> P3 D+
- Y1 pad 1: XTAL2 -> XTAL1
- Y1 pad 2: XTAL1 -> GND
- Y1 pad 3: (no net) -> XTAL2
- Y1 pad 4: (no net) -> GND
Routing:
- net +5V: track 0.00 -> 170.9 mm, vias 0 -> 4
- net P3 D-: track 0.00 -> 51.3 mm
- net P3 D+: track 0.00 -> 49.2 mm, vias 0 -> 2
- net GND: track 0.00 -> 33.4 mm
- net P2 D+: track 0.00 -> 30.5 mm
- net P2 D-: track 0.00 -> 28.6 mm
- net P1 D+: track 0.00 -> 14.2 mm
- net Net-(F4-Pad1): track 0.00 -> 14.1 mm
- net P1 D-: track 0.00 -> 14.1 mm, vias 0 -> 2
- net Net-(F2-Pad1): track 0.00 -> 7.92 mm
- net Net-(F3-Pad1): track 0.00 -> 7.91 mm
- net Net-(J2-Pad3): track 0.00 -> 7.49 mm
- net Net-(J2-Pad2): track 0.00 -> 7.43 mm, vias 0 -> 1
- net Net-(J3-Pad3): track 0.00 -> 7.17 mm
- net Net-(J3-Pad2): track 0.00 -> 7.15 mm, vias 0 -> 1
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- added copper zone on B.Cu, net GND
- added copper zone on F.Cu, net GND

Commit message: layout done, saving for 0805 change
Parts:
- removed R7: 5k, Resistor_SMD:R_0805_2012Metric
- removed RESET1: RESET, colonDcustom:Pushbutton_TH_6x6
- added C11: .1u, Capacitor_SMD:C_0402_1005Metric, F.Cu at (101.5, 72.5)
- added C12: .1u, Capacitor_SMD:C_0402_1005Metric, F.Cu at (89.9, 77.7)
- added C13: .1u, Capacitor_SMD:C_0402_1005Metric, F.Cu at (99.5, 77.2)
- added C14: 4.7u, Capacitor_SMD:C_0603_1608Metric, F.Cu at (100.5, 65.5)
- added C15: .1u, Capacitor_SMD:C_0402_1005Metric, F.Cu at (101.5, 73.5)
- added C16: .1u, Capacitor_SMD:C_0402_1005Metric, F.Cu at (91.5, 67.0)
- added C17: 4.7u, Capacitor_SMD:C_0603_1608Metric, F.Cu at (102.2, 66.0)
- added C19: 1u, Capacitor_SMD:C_0603_1608Metric, F.Cu at (128.5, 96.0)
- added FB1: 600, Resistor_SMD:R_0603_1608Metric, F.Cu at (109.5, 49.1)
- C1, C7: footprint Capacitor_SMD:C_0805_2012Metric -> Capacitor_SMD:C_0603_1608Metric
- C10, C4, C8, C9: value 1u -> .1u; footprint Capacitor_SMD:C_0805_2012Metric -> Capacitor_SMD:C_0402_1005Metric
- C2, C3: value 18p -> 8p; footprint Capacitor_SMD:C_0805_2012Metric -> Capacitor_SMD:C_0402_1005Metric
- C5: value .1u -> 1u; footprint Capacitor_SMD:C_0805_2012Metric -> Capacitor_SMD:C_0603_1608Metric
- C6: footprint Capacitor_SMD:C_0805_2012Metric -> Capacitor_SMD:C_0402_1005Metric
- F1: value 500m -> 1; footprint Fuse:Fuse_0805_2012Metric -> Fuse:Fuse_0603_1608Metric
- F2, F3, F4: value 400m -> 900m; footprint Fuse:Fuse_0805_2012Metric -> Fuse:Fuse_0603_1608Metric
- J1: footprint Connector_USB:USB_C_Receptacle_GCT_USB4085 -> colonDcustom:USB_C_Receptacle_HRO_TYPE-C-31-M-12
- J2: footprint Connector_USB:USB3_A_Molex_48393-001 -> colonDcustom:USB_A_CONNFLY_DS1095-WNR0
- J3: value USB A, Port 2 -> USB C 2.0, Port 2; footprint Connector_USB:USB3_A_Molex_48393-001 -> colonDcustom:USB_C_Receptacle_HRO_TYPE-C-31-M-12
- J4: value USB C 2.0, Port 3 -> USB A, Port 3; footprint Connector_USB:USB_C_Receptacle_GCT_USB4085 -> colonDcustom:USB_A_CONNFLY_DS1095-WNR0
- R1: value 50k -> 5k1; footprint Resistor_SMD:R_0805_2012Metric -> Resistor_SMD:R_0603_1608Metric
- R2: value 10k -> 5k1; footprint Resistor_SMD:R_0805_2012Metric -> Resistor_SMD:R_0603_1608Metric
- R3: value 100k -> 12k 1%; footprint Resistor_SMD:R_0805_2012Metric -> Resistor_SMD:R_0603_1608Metric
- R4: value 5k -> 50k; footprint Resistor_SMD:R_0805_2012Metric -> Resistor_SMD:R_0603_1608Metric
- R5: value 5k -> 100k; footprint Resistor_SMD:R_0805_2012Metric -> Resistor_SMD:R_0603_1608Metric
- R6: value 5k -> 10k; footprint Resistor_SMD:R_0805_2012Metric -> Resistor_SMD:R_0603_1608Metric
- Y1: value Crystal_GND24 -> 24M; footprint Crystal:Crystal_SMD_0603-4Pin_6.0x3.5mm -> Crystal:Crystal_SMD_2016-4Pin_2.0x1.6mm
- moved C5 128.5 mm to (102.1, 107.1), turned to -90 degrees
- moved C6 117.5 mm to (92.8, 78.1), turned to -90 degrees
- moved R4 112.0 mm to (97.3, 61.8)
- moved R2 104.6 mm to (103.5, 47.4), turned to 180 degrees
- moved C4 101.1 mm to (95.8, 66.8)
- moved R3 99.7 mm to (88.4, 77.0), turned to -90 degrees
- moved U3 97.7 mm to (106.3, 105.9)
- moved R6 96.6 mm to (94.8, 65.0), turned to 0 degrees
- moved F3 95.9 mm to (103.7, 107.1)
- moved J3 95.1 mm to (106.4, 115.8)
- moved R5 90.2 mm to (97.3, 63.4), turned to 0 degrees
- moved C8 83.7 mm to (92.5, 66.9), turned to 90 degrees
- moved C9 83.1 mm to (96.8, 67.2), turned to 90 degrees
- moved R1 79.5 mm to (103.5, 49.1)
- moved C10 78.6 mm to (91.5, 77.7)
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Connections:
- C10 pad 1: +5V -> VDD33
- C4 pad 1: +5V -> GND
- C4 pad 2: GND -> RESET
- C8 pad 1: VDD12 -> VDD33
- F1 pad 2: +5V -> Net-(F1-Pad2)
- J1 pad A5: unconnected-(J1-PadA5) -> Net-(J1-PadA5)
- J1 pad A8: GND -> unconnected-(J1-PadA8)
- J1 pad B5: unconnected-(J1-PadB5) -> Net-(J1-PadB5)
- J1 pad B8: GND -> unconnected-(J1-PadB8)
- J1 pad S1: GND -> unconnected-(J1-PadS1)
- J2 pad 5: GND -> unconnected-(J2-Pad5)
- R1 pad 1: +5V -> Net-(J1-PadA5)
- R1 pad 2: +3V3 -> GND
- R2 pad 1: +5V -> Net-(J1-PadB5)
- R2 pad 2: RESET -> GND
- R3 pad 1: +3V3 -> Net-(R3-Pad1)
- R4 pad 2: OCS1 -> +3V3
- R5 pad 1: +5V -> +3V3
- R5 pad 2: OCS2 -> GND
- R6 pad 1: +5V -> +3V3
- R6 pad 2: OCS3 -> RESET
- U1 pad 10: unconnected-(U1-Pad10) -> P4 D-
- U1 pad 11: unconnected-(U1-Pad11) -> P4 D+
- U1 pad 16: OCS1 -> unconnected-(U1-Pad16)
- U1 pad 20: OCS2 -> unconnected-(U1-Pad20)
- U1 pad 24: SPI_DI -> unconnected-(U1-Pad24)
- U1 pad 25: SPI_CS -> unconnected-(U1-Pad25)
- U1 pad 26: SPI_DO -> unconnected-(U1-Pad26)
- U1 pad 27: SPI_CLK -> unconnected-(U1-Pad27)
- U1 pad 28: OCS3 -> unconnected-(U1-Pad28)
- U1 pad 30: OCS4 -> unconnected-(U1-Pad30)
- U1 pad 31: I2C_SDA -> unconnected-(U1-Pad31)
- U1 pad 32: unconnected-(U1-Pad32) -> VDD33
- U1 pad 33: I2C_SCL -> unconnected-(U1-Pad33)
- U1 pad 38: unconnected-(U1-Pad38) -> VDD12
- U1 pad 46: unconnected-(U1-Pad46) -> Net-(R3-Pad1)
- U2 pad 1: Net-(J2-Pad3) -> Net-(J2-Pad2)
- U2 pad 3: Net-(J2-Pad2) -> Net-(J2-Pad3)
- U2 pad 4: P1 D- -> P1 D+
- U2 pad 6: P1 D+ -> P1 D-
- U3 pad 1: Net-(J3-Pad3) -> Net-(J3-PadA7)
- U3 pad 3: Net-(J3-Pad2) -> Net-(J3-PadA6)
- U3 pad 4: P3 D- -> P2 D+
- U3 pad 6: P3 D+ -> P2 D-
- U4 pad 1: Net-(J4-PadA7) -> Net-(J4-Pad2)
- U4 pad 3: Net-(J4-PadA6) -> Net-(J4-Pad3)
- U4 pad 4: P2 D+ -> P3 D+
- U4 pad 6: P2 D- -> P3 D-
Routing:
- net +5V: track 170.9 -> 35.2 mm, vias 4 -> 14
- net P3 D-: track 51.3 -> 0.00 mm
- net VDD33: track 0.00 -> 50.5 mm, vias 0 -> 6
- net P3 D+: track 49.2 -> 0.00 mm, vias 2 -> 0
- net P2 D+: track 30.5 -> 0.00 mm
- net P2 D-: track 28.6 -> 0.00 mm
- net VDD12: track 1.62 -> 28.6 mm, vias 0 -> 3
- net Net-(J1-PadA5): track 0.00 -> 18.4 mm, vias 0 -> 2
- net unconnected-(J3-PadS1): track 0.00 -> 17.1 mm
- net unconnected-(J1-PadS1): track 0.00 -> 17.0 mm
- net P1 D+: track 14.2 -> 0.00 mm
- net P1 D-: track 14.1 -> 0.00 mm, vias 2 -> 0
- net Net-(F4-Pad1): track 14.1 -> 2.73 mm
- net RESET: track 0.00 -> 8.65 mm
- net Net-(J3-PadA7): track 0.00 -> 8.25 mm
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- added copper zone on In2.Cu, net +5V
- added copper zone on In1.Cu, net GND
- removed copper zone on B.Cu, net GND
- removed copper zone on F.Cu, net GND
Other:
- board outline added: 80.4 x 80.6 mm
- copper layers 2 -> 4
- rule pad_to_mask_clearance: 0 -> 0.05

Commit message: V1.0
Parts:
- C1, C14, C17, C19, C5, C7: footprint Capacitor_SMD:C_0603_1608Metric -> Capacitor_SMD:C_0805_2012Metric
- C10, C11, C12, C13, C15, C16, C2, C3, C4, C6, C8, C9: footprint Capacitor_SMD:C_0402_1005Metric -> Capacitor_SMD:C_0805_2012Metric
- F1, F2, F3, F4: footprint Fuse:Fuse_0603_1608Metric -> Fuse:Fuse_0805_2012Metric
- FB1, R1, R2, R3, R4, R5, R6: footprint Resistor_SMD:R_0603_1608Metric -> Resistor_SMD:R_0805_2012Metric
- Y1: footprint Crystal:Crystal_SMD_2016-4Pin_2.0x1.6mm -> Crystal:Crystal_SMD_3225-4Pin_3.2x2.5mm
- moved C9 16.6 mm to (109.6, 56.6)
- moved R4 15.6 mm to (108.9, 51.4)
- moved C8 15.4 mm to (102.7, 55.4)
- moved R5 15.3 mm to (108.9, 53.5)
- moved C17 15.1 mm to (113.9, 56.6)
- moved R6 14.9 mm to (105.9, 55.1), turned to -90 degrees
- moved C14 14.4 mm to (111.7, 56.6)
- moved C16 14.3 mm to (100.6, 56.0)
- moved C4 12.9 mm to (105.9, 58.7)
- moved C11 9.79 mm to (107.5, 64.8)
- moved F1 9.26 mm to (115.6, 40.4)
- moved J1 9.26 mm to (112.4, 33.7)
- moved R2 9.26 mm to (109.6, 40.4)
- moved R1 9.03 mm to (109.6, 42.5)
- moved FB1 9.03 mm to (115.7, 42.5)
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Routing:
- net P3 D+: track 0.00 -> 69.9 mm, vias 0 -> 2
- net P3 D-: track 0.00 -> 69.6 mm, vias 0 -> 2
- net P2 D+: track 0.00 -> 55.5 mm, vias 0 -> 2
- net P2 D-: track 0.00 -> 55.3 mm, vias 0 -> 2
- net UP D+: track 3.28 -> 40.5 mm
- net UP D-: track 3.39 -> 39.8 mm
- net P1 D+: track 0.00 -> 35.2 mm
- net P1 D-: track 0.00 -> 35.1 mm
- net +5V: track 35.2 -> 68.6 mm, vias 14 -> 12
- net unconnected-(J2-Pad5): track 0.00 -> 13.4 mm
- net unconnected-(J4-Pad5): track 0.00 -> 13.1 mm
- net VDD33: track 50.5 -> 62.7 mm, vias 6 -> 5
- net GND: track 39.3 -> 48.2 mm, vias 51 -> 49
- net +3V3: track 10.00 -> 18.1 mm
- net Net-(R3-Pad1): track 5.48 -> 13.0 mm
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Other:
- board size 80.4 x 80.6 mm -> 80.8 x 84.6 mm
- rule pad_to_mask_clearance: 0.05 -> 0
- board text added: ":D designs Anduril USB Hub v1.0 Dec 2022"
- board text added: "To the amazing employees of Anduril Industries Dec 2022"
- board text added: "USB 2.0 1A Input Fuse 900mA Output Fuse per port"

Commit message: v1.1 WIP
Parts:
- added C1: .1u, Capacitor_SMD:C_0805_2012Metric, F.Cu at (119.8, 35.1)
- added C22: .1u, Capacitor_SMD:C_0805_2012Metric, F.Cu at (136.2, 91.8)
- added C3: .1u, Capacitor_SMD:C_0805_2012Metric, F.Cu at (99.8, 107.5)
- added C8: .1u, Capacitor_SMD:C_0805_2012Metric, F.Cu at (117.4, 102.8)
- added R10: 1M, Resistor_SMD:R_0805_2012Metric, F.Cu at (137.4, 93.8)
- added R4: 1M, Resistor_SMD:R_0805_2012Metric, F.Cu at (119.8, 37.6)
- added R5: 1M, Resistor_SMD:R_0805_2012Metric, F.Cu at (101.0, 105.7)
- added R9: 1M, Resistor_SMD:R_0805_2012Metric, F.Cu at (117.4, 105.0)
- added U1: USBLC6-2SC6, Package_TO_SOT_SMD:SOT-23-6, F.Cu at (111.9, 41.7)
- F1: value 1 -> 500m
- F2, F3, F4: value 900m -> 400m
- moved R2 3.04 mm to (106.6, 40.4)
- moved R1 3.03 mm to (106.6, 42.4)
- moved F1 1.16 mm to (116.8, 40.4)
- moved FB1 1.15 mm to (116.8, 42.5)
- moved C10 1.12 mm to (116.8, 44.6)
- renumbered C7 to C10, C8 to C11, C9 to C12, C10 to C13, C11 to C14, C12 to C15, C13 to C16, C14 to C17, C15 to C18, C16 to C19, C1 to C2, C17 to C20, C19 to C21, C2 to C4, C3 to C5, C4 to C6, C5 to C7, C6 to C9, R4 to R6, R5 to R7, R6 to R8, U1 to U2, U2 to U3, U3 to U4, U4 to U5
Connections:
- J1 pad A6: UP D+ -> Net-(J1-PadA6)
- J1 pad A7: UP D- -> Net-(J1-PadA7)
- J1 pad B6: UP D+ -> Net-(J1-PadA6)
- J1 pad B7: UP D- -> Net-(J1-PadA7)
- J1 pad S1: unconnected-(J1-PadS1) -> Net-(C1-Pad1)
- J2 pad 5: unconnected-(J2-Pad5) -> Net-(C3-Pad1)
- J3 pad S1: unconnected-(J3-PadS1) -> Net-(C8-Pad1)
- J4 pad 5: unconnected-(J4-Pad5) -> Net-(C22-Pad1)
Routing:
- net Net-(C1-Pad1): track 0.00 -> 25.4 mm
- net Net-(C8-Pad1): track 0.00 -> 23.6 mm
- net Net-(C22-Pad1): track 0.00 -> 20.2 mm
- net Net-(C3-Pad1): track 0.00 -> 19.1 mm
- net unconnected-(J3-PadS1): track 17.1 -> 0.00 mm
- net unconnected-(J1-PadS1): track 17.0 -> 0.00 mm
- net GND: track 48.2 -> 63.2 mm, vias 49 -> 59
- net unconnected-(J2-Pad5): track 13.4 -> 0.00 mm
- net unconnected-(J4-Pad5): track 13.1 -> 0.00 mm
- net UP D+: track 40.5 -> 31.8 mm
- net UP D-: track 39.8 -> 31.9 mm
- net Net-(J1-PadA6): track 0.00 -> 6.43 mm
- net VCC: track 10.5 -> 16.2 mm
- net Net-(J1-PadA7): track 0.00 -> 5.05 mm
- net Net-(J1-PadB5): track 2.74 -> 4.92 mm
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Other:
- board text added: "Anduril USB Hub v1.1 :D designs github.com/colonDdesigns Dec 2022"
- board text added: "USB 2.0 500mA Input fuse 350mA Output fuse per port"
- board text removed: ":D designs Anduril USB Hub v1.0 Dec 2022"
- board text removed: "USB 2.0 1A Input Fuse 900mA Output Fuse per port"
