File: v1.1/electrical/Anduril USB Hub.kicad_sch (KiCad schematic)
At the start: 47 parts, among them J1 USB C 2.0, Upstream, J2 USB A, Port 1, J3 USB C 2.0, Port 2, J4 USB A, Port 3, U1 USBLC6-2SC6, U2 USB4604-1080HN, U3 USBLC6-2SC6, U4 USBLC6-2SC6, U5 USBLC6-2SC6, Y1 24M

Commit message: readme updates
Other:
- note added: "Anduril USB Hub v1.1"
- note removed: "Anduril USB Hub"
Changed lines of the file:
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@@
     (effects (font (size 3 3)) (justify left bottom))
   )
-  (text "Anduril USB Hub" (at 309.88 278.13 0)
+  (text "Anduril USB Hub v1.1" (at 309.88 278.13 0)
     (effects (font (size 2.5 2.5) (thickness 0.5) bold) (justify left bottom))
   )
